Commit message: chunkbot on ros humble

File: description/robot.urdf.xacro (robot description, xacro)
@@ -1,8 +1,5 @@
 <?xml version="1.0"?>
 <robot xmlns:xacro="http://www.ros.org/wiki/xacro"  name="robot">
-    <xacro:include filename="robot_core.xacro" />
-    <xacro:include filename="gazebo_control.xacro"/>
-    <xacro:include filename="ros2_control.xacro"/>
-    <xacro:include filename="lidar.xacro"/>
-    <xacro:include filename= "camera.xacro"/>
+    <!-- Example link -->
+    <link name="base_link"></link>
 </robot>

Commit message: Revert "urdf setup"

File: description/robot.urdf.xacro (robot description, xacro)
@@ -1,4 +1,5 @@
 <?xml version="1.0"?>
 <robot xmlns:xacro="http://www.ros.org/wiki/xacro"  name="robot">
-    <xacro:include filename="robot_core.xacro" />
+    <!-- Example link -->
+    <link name="base_link"></link>
 </robot>

Commit message: Revert "chunkbot on ros humble"

File: description/robot.urdf.xacro (robot description, xacro)
@@ -1,5 +1,8 @@
 <?xml version="1.0"?>
 <robot xmlns:xacro="http://www.ros.org/wiki/xacro"  name="robot">
-    <!-- Example link -->
-    <link name="base_link"></link>
+    <xacro:include filename="robot_core.xacro" />
+    <xacro:include filename="gazebo_control.xacro"/>
+    <xacro:include filename="ros2_control.xacro"/>
+    <xacro:include filename="lidar.xacro"/>
+    <xacro:include filename= "camera.xacro"/>
 </robot>
